File: fluke_884x_continuity_buzzer.kicad_sch (KiCad schematic)
At the start: 70 parts, among them J2 Conn_01x02, J203 16 pin DIP socket, J204 16 pin DIP socket, J3 USB_B_Micro, P203 16 pin DIP plug, P204 16 pin DIP plug, U1 NCP1117-3.3_SOT223, U2 W25Q128JVS, U3 RP2040, Y1 ABLS-12.000MHZ-B4-T

Commit message: Added LCSC refs
Parts:
- C1, C2, C3: LCSC (none) -> C15850
- C10, C11, C12, C14, C16, C17, C4, C5, C6, C8: LCSC (none) -> C1525
- C13, C15: LCSC (none) -> C52923
- C7, C9: LCSC (none) -> C1557
- D1: LCSC (none) -> C282361
- D2, D3, D4, D5, D6, D7, D8: LCSC (none) -> C5240639
- J203, J204: LCSC (none) -> C157594
- J3: footprint RP2040_minimal:USB_Micro-B_Amphenol_10103594-0001LF_Horizontal_modified -> Connector_USB:USB_Micro-B_Amphenol_10118194_Horizontal; LCSC (none) -> C132563
- P203, P204: now not fitted; now left out of the parts list
- R1, R10, R11, R12, R13, R14, R15, R16, R17, R19, R2, R21, R3, R4, R5, R6, R7, R8, R9: LCSC (none) -> C25790
- R18, R20, R22, R23, R24, R25, R26: LCSC (none) -> C25756
- R27: now not fitted
- R28, R29: LCSC (none) -> C11702
- R30, R31: LCSC (none) -> C25156
- TP1, TP2, TP3: now left out of the parts list
- U1: value NCP1117-3.3_SOT223 -> AZ117EH-3.3; LCSC (none) -> C108494
- U2: LCSC (none) -> C97521
- U3: LCSC (none) -> C2040
- Y1: LCSC (none) -> C326543
Other:
- note added: "Make sure C13 is close to pin 45 of RP2040"
- note added: "Make sure C15 is close to pin 44 of RP2040"
- note added: "Make sure R30 and R31 are close to RP2040"
- note removed: "Make sure C3 is close to pin 45 of RP2040"
- note removed: "Make sure C6 is close to pin 44 of RP2040"
- note removed: "Make sure R20 and R21 are close to RP2040"

Commit message: Updated text; fixed silk
Parts:
- J2: LCSC (none) -> C2685154
- LS1: footprint Buzzer_Beeper:Buzzer_12x9.5RM7.6 -> RP2040_minimal:Buzzer_17x9RM10; LCSC (none) -> C360609
Changed lines of the file:
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@@
 			)
 		)
-		(property "Footprint" "Buzzer_Beeper:Buzzer_12x9.5RM7.6"
+		(property "Footprint" "RP2040_minimal:Buzzer_17x9RM10"
 			(at 278.511 227.33 0)
 			(effects
@@
 			)
 		)
-		(property "Field-1" ""
+		(property "LCSC" "C360609"
 			(at 279.4 226.06 0)
 			(effects
@@
 			)
 		)
-		(property "Field-1" ""
+		(property "LCSC" "C2685154"
 			(at 212.725 56.515 0)
 			(effects
