File: hardware/fluke_884x_continuity_buzzer.kicad_sch (KiCad schematic)
At the start: 64 parts, among them J2 Conn_01x02, J203 16 pin DIP socket, J204 16 pin DIP socket, J3 USB_B_Micro, P203 16 pin DIP plug, P204 16 pin DIP plug, U1 AZ117EH-3.3, U2 W25Q128JVS, U3 RP2040, U4 umw_78l05_sot23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

Commit message: Removed bus buffer
Parts:
- removed R22: 10k, Resistor_SMD:R_0402_1005Metric, symbol Device:R
- removed U5: SN74LVC8T245PW, Package_SO:TSSOP-24_4.4x7.8mm_P0.65mm, symbol Logic_LevelTranslator:SN74AVC8T245PW
Other:
- note removed: "U5 allows watching or driving the (5V logic) keypad RL0-RL6 lines. DIR H, ~{OE} L: A->B DIR L, ~{OE} L: B->A ~{OE} H: both sides Hi-Z"
