File: hardware/fluke_884x_continuity_buzzer.kicad_sch (KiCad schematic)
At the start: 63 parts, among them J2 Conn_01x02, J203 16 pin DIP socket, J204 16 pin DIP socket, J3 USB_B_Micro, P203 16 pin DIP plug, P204 16 pin DIP plug, U1 AZ117EH-3.3, U2 W25Q128JVS, U3 RP2040, Y1 ABLS-12.000MHZ-B4-T

Commit message: Exclude plugs and USB BOOT header from production
Parts:
- J2, P203, P204: now not fitted; now left out of the parts list
Changed lines of the file:
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@@
 		(unit 1)
 		(exclude_from_sim no)
-		(in_bom yes)
+		(in_bom no)
 		(on_board yes)
-		(dnp no)
+		(dnp yes)
 		(property "Reference" "J2"
 			(at 212.09 53.34 0)
@@
 		(unit 1)
 		(exclude_from_sim no)
-		(in_bom yes)
+		(in_bom no)
 		(on_board yes)
-		(dnp no)
+		(dnp yes)
 		(property "Reference" "P204"
 			(at 101.092 30.734 0)
@@
 		(unit 1)
 		(exclude_from_sim no)
-		(in_bom yes)
+		(in_bom no)
 		(on_board yes)
-		(dnp no)
+		(dnp yes)
 		(property "Reference" "P203"
 			(at 60.96 31.242 0)

Commit message: Change to using external GND connection
Parts:
- removed R27: DNF, Resistor_SMD:R_0402_1005Metric, symbol Device:R
- added TP4: GND_IN, TestPoint:TestPoint_THTPad_D2.0mm_Drill1.0mm, symbol Connector:TestPoint
Connections:
- net GND: now also TP4.1; no longer J203.16 (Pin_16), P203.1 (Pin_1)
- new net GND2: J203.16 (Pin_16), P203.1 (Pin_1)
Other:
- note removed: "Crystal"
- note removed: "F1-F2 are from a 4.5VAC transformer whose center-tap is tied to +5V. The Pxx and Gxx lines are 30V logic. All 19 of these lines are clamped to 3.3V using the 200k resistors R1-R19 and their associated Schottky diodes. The S0-S2 lines are inverted, current-sinking, 5V versions of G0-G2 used for scanning the key matrix columns. Since these duplicate G0-G2, we don't bother watching them also. The RL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"
- note removed: "Flash"
- moved on the sheet: C1, C10, C11, C12, C13, C14, C15, C16, C17, C18, C2, C3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
