File: combo_board/combo_board.kicad_sch (KiCad schematic)
At the start: 63 parts, among them J2 Conn_01x02, J203 16 pin DIP socket, J204 16 pin DIP socket, J3 USB_B_Micro, P203 16 pin DIP plug, P204 16 pin DIP plug, U1 AZ117EH-3.3, U2 W25Q128JVS, U3 RP2040, Y1 ABLS-12.000MHZ-B4-T

Commit message: Ordered from JLCPCB; add combo board project
Parts:
- removed C18: 220uF, Capacitor_THT:C_Radial_D6.3mm_H11.0mm_P2.50mm, symbol Device:C_Polarized_US
- removed D1: BAS40-05W, Package_TO_SOT_SMD:SOT-323_SC-70, symbol misc:bas40-05w_split
- removed J203, J204: 16 pin DIP socket, Package_DIP:DIP-16_W7.62mm_Socket, symbol Connector:Conn_01x16_Socket
- removed P203, P204: 16 pin DIP plug, RP2040_minimal:DIP-16_W7.62mm, symbol Connector:Conn_01x16_Pin
- added TP5: 5V_IN, TestPoint:TestPoint_THTPad_D3.0mm_Drill1.5mm, symbol Connector:TestPoint
Connections:
- net EXT_5V: now reaches C1.1, D2.3 (K), D2.3 (K), U1.3 (VI)
- net EXT_5V: now also TP5.1
Other:
- added sheet Connections (connections.kicad_sch)
- added sheet Keyboard and Display (keyboard_and_display.kicad_sch)
- note added: "Continuity Buzzer"
- note removed: "Fluke 884x Continuity Buzzer"
- title: Fluke 884x Continuity Buzzer -> Fluke 884x Display/Keypad/Continuity Buzzer
- moved on the sheet: C1, C10, C11, C12, C13, C14, C15, C16, C17, C2, C3, C4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

Commit message: Moved GND, +5V inputs to L Rear of board
Parts:
- J3: footprint RP2040_minimal:USB_Micro-B_Amphenol_10118194_Horizontal -> Connector_USB:USB_Micro-B_Molex-105133-0001
Changed lines of the file:
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@@
 			)
 		)
-		(property "Footprint" "RP2040_minimal:USB_Micro-B_Amphenol_10118194_Horizontal"
+		(property "Footprint" "Connector_USB:USB_Micro-B_Molex-105133-0001"
 			(at 312.42 139.7 0)
 			(effects

Commit message: Got JLCPCB order ready
Parts:
- TP2, TP3: now left out of the parts list
Changed lines of the file:
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@@
 		(unit 1)
 		(exclude_from_sim no)
-		(in_bom yes)
+		(in_bom no)
 		(on_board yes)
 		(dnp no)
@@
 		(unit 1)
 		(exclude_from_sim no)
-		(in_bom yes)
-		(on_board yes)
-		(dnp no)
+		(in_bom no)
+		(on_board yes)
+		(dnp no)
