File: combo_board/combo_board.kicad_pcb (KiCad board)
At the start: 4 copper layers, 188 x 71.8 mm, 84 parts, among them J2 Conn_01x02, J203 16 pin DIP socket, J204 16 pin DIP socket, J3 USB_B_Micro, SW1 SW_Push_45deg, SW10 SW_Push_45deg, SW11 SW_Push_45deg, SW12 SW_Push_45deg, SW13 SW_Push_45deg, SW14 SW_Push_45deg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

Commit message: Move GND terminal to clear chassis
Parts:
- moved TP4 12.4 mm to (158.1, 102.4)
Routing:
- net EXT_5V: track 95.5 -> 98.0 mm
Other:
- board text added: "GND"
Changed lines of the file:
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@@
 	(title_block
 		(title "Fluke 884x Keypad/Display/Continuity Buzzer")
-		(date "2024-09-27")
-		(rev "1")
+		(date "2024-10-18")
+		(rev "2")
 		(company "Ned Konz")
 	)
@@
 	(footprint "TestPoint:TestPoint_THTPad_D3.0mm_Drill1.5mm"
 		(layer "B.Cu")
-		(at 169.15 96.737317 180)
+		(at 158.07 102.357317 180)
 		(descr "THT pad as test Point, diameter 3.0mm, hole diameter 1.5mm")
 		(tags "test point THT pad")
@@
 		(tags "Test Point")
 		(property "Reference" "TP1"
-			(at -1.57 -2.35 0)
+			(at -4.16 -1.41 0)
 			(layer "B.SilkS")
 			(effects
@@
 			(justify left bottom mirror)
 		)
-		(render_cache "(C) Ned Konz 2024\nRev. 1" -0
+		(render_cache "(C) Ned Konz 2024\nRev. 2" -0
 			(polygon
 				(pts
@@
 			(polygon
 				(pts
-					(xy 45.664487 96.664002) (xy 45.664487 96.056814) (xy 45.703939 96.087783) (xy 45.748812 96.120688)
-					(xy 45.796142 96.151657) (xy 45.842374 96.176046) (xy 45.891632 96.188949) (xy 45.939024 96.171858)
-					(xy 45.948541 96.16306) (xy 45.971439 96.119691) (xy 45.972965 96.10322) (xy 45.959639 96.05573)
-					(xy 45.949274 96.045335) (xy 45.906665 96.019002) (xy 45.868918 95.999905) (xy 45.825364 95.97734)
-					(xy 45.783089 95.951542) (xy 45.74086 95.919576) (xy 45.737759 95.916863) (xy 45.702451 95.882562)
-					(xy 45.670165 95.845239) (xy 45.650321 95.818677) (xy 45.62163 95.778566) (xy 45.59903 95.749801)
-					(xy 45.550181 95.735635) (xy 45.502503 95.750181) (xy 45.485945 95.766409) (xy 45.465375 95.813273)
-					(xy 45.462009 95.849452) (xy 45.462009 96.636891) (xy 45.46559 96.686527) (xy 45.481504 96.736735)
-					(xy 45.519299 96.773819) (xy 45.563859 96.782948) (xy 45.61152 96.772185) (xy 45.636887 96.752418)
-					(xy 45.659932 96.706519)
+					(xy 45.725547 96.59537) (xy 45.381409 96.59537) (xy 45.331461 96.60117) (xy 45.294459 96.618573)
+					(xy 45.266118 96.660759) (xy 45.263684 96.682076) (xy 45.27756 96.72952) (xy 45.288353 96.742648)
+					(xy 45.33347 96.764907) (xy 45.361381 96.767317) (xy 45.866964 96.767317) (xy 45.915812 96.759806)
+					(xy 45.952937 96.737275) (xy 45.979594 96.695429) (xy 45.983956 96.6662) (xy 45.972328 96.616356)
+					(xy 45.964905 96.599033) (xy 45.940701 96.556216) (xy 45.922651 96.534065) (xy 45.883433 96.493379)
+					(xy 45.845922 96.455312) (xy 45.810117 96.419862) (xy 45.771286 96.382554) (xy 45.757299 96.369445)
+					(xy 45.719112 96.334549) (xy 45.681412 96.301973) (xy 45.651542 96.279075) (xy 45.612455 96.249216)
+					(xy 45.573626 96.214381) (xy 45.559218 96.199452) (xy 45.526978 96.159274) (xy 45.503531 96.118363)
+					(xy 45.487624 96.069832) (xy 45.48448 96.037519) (xy 45.492303 95.988231) (xy 45.504508 95.962048)
+					(xy 45.53668 95.924867) (xy 45.558485 95.910513) (xy 45.606205 95.894144) (xy 45.633468 95.89195)
+					(xy 45.683471 95.899416) (xy 45.730209 95.924874) (xy 45.765186 95.963695) (xy 45.76829 95.968398)
+					(xy 45.788024 96.016112) (xy 45.791004 96.024574) (xy 45.810994 96.070873) (xy 45.829106 96.098335)
+					(xy 45.871331 96.123077) (xy 45.893831 96.125202) (xy 45.94124 96.112206) (xy 45.956357 96.100045)
+					(xy 45.979299 96.054797) (xy 45.98127 96.032146) (xy 45.975835 95.98177) (xy 45.960869 95.932658)
+					(xy 45.959532 95.929319) (xy 45.936231 95.884433) (xy 45.904795 95.84338) (xy 45.894319 95.832355)
+					(xy 45.855206 95.799813) (xy 45.812376 95.774711) (xy 45.78441 95.762257) (xy 45.73611 95.7471)
+					(xy 45.687643 95.738781) (xy 45.634835 95.735661) (xy 45.629316 95.735635) (xy 45.577887 95.737757)
+					(xy 45.524665 95.745216) (xy 45.47635 95.758047) (xy 45.446866 95.769584) (xy 45.403067 95.794865)
+					(xy 45.364635 95.827659) (xy 45.359916 95.832599) (xy 45.328356 95.872713) (xy 45.304203 95.918409)
+					(xy 45.301542 95.924923) (xy 45.28664 95.974783) (xy 45.280862 96.02636) (xy 45.280781 96.033367)
+					(xy 45.285003 96.0869) (xy 45.297668 96.137284) (xy 45.318777 96.184521) (xy 45.324012 96.19359)
+					(xy 45.351022 96.235393) (xy 45.381063 96.274268) (xy 45.411451 96.305698) (xy 45.448938 96.338714)
+					(xy 45.489914 96.373628) (xy 45.528195 96.405698) (xy 45.558974 96.431238) (xy 45.60097 96.466685)
+					(xy 45.641381 96.502672) (xy 45.677172 96.537392) (xy 45.70039 96.563129)
 				)
 			)
@@
 	)
 	(gr_text "GND_IN"
-		(at 176.06 94.897317 -0)
+		(at 160.43 100.237317 -0)
 		(layer "B.SilkS")
 		(effects
@@
 	)
 	(gr_text "5V_IN"
-		(at 175.75 103.067317 0)
+		(at 171.66 100.317317 0)
 		(layer "B.SilkS")
 		(effects
@@
 		)
 	)
+	(gr_text "GND"
+		(at 40.4 104.087317 0)
+		(layer "B.SilkS")
+		(effects
+			(font
+				(size 1 1)
+				(thickness 0.15)
+			)
+			(justify left bottom mirror)
+		)
+	)
 	(gr_text "BRN"
 		(at 31.44 128.677317 0)
@@
 	)
 	(segment
+		(start 128.69 101.807317)
+		(end 128.69 101.187317)
+		(width 1)
+		(layer "B.Cu")
+		(net 15)
+	)
+	(segment
 		(start 118.52 99.557317)
 		(end 118.52 100.437317)
@@
 	)
 	(segment
+		(start 165.91 99.217317)
+		(end 169.21 102.517317)
+		(width 1)
+		(layer "B.Cu")
+		(net 15)
+	)
+	(segment
 		(start 88.25 99.547317)
 		(end 88.53 94.657317)
@@
 	)
 	(segment
-		(start 169.21 102.517317)
-		(end 168.5 101.807317)
+		(start 118.52 100.437317)
+		(end 118.7 100.617317)
 		(width 1)
 		(layer "B.Cu")
@@
 	)
 	(segment
-		(start 118.52 100.437317)
-		(end 118.7 100.617317)
+		(start 128.69 101.187317)
+		(end 130.66 99.217317)
 		(width 1)
 		(layer "B.Cu")
@@
 	)
 	(segment
-		(start 168.5 101.807317)
-		(end 128.69 101.807317)
+		(start 130.66 99.217317)
+		(end 165.91 99.217317)
 		(width 1)
 		(layer "B.Cu")
